Commit message: temporal filter changes with new library files

File: realsense_ros_camera/urdf/_r410.urdf.xacro (robot description, xacro)
@@ -7,4 +7,5 @@
 -->
 <robot name="sensor_r410" xmlns:xacro="http://ros.org/wiki/xacro">
+  <xacro:include filename="$(find industrial_extrinsic_cal)/urdf/calibration_transform_macro.xacro"/>
   <xacro:property name="M_PI" value="3.1415926535897931" />
   <!-- The following values are approximate, and the camera node
@@ -29,10 +30,10 @@
   <xacro:macro name="sensor_r410" params="parent *origin">
     <!-- camera body, with origin at bottom screw mount -->
-    <joint name="camera_joint" type="fixed">
+    <joint name="realsense_joint" type="fixed">
       <xacro:insert_block name="origin" />
       <parent link="${parent}"/>
-      <child link="camera_link" />
+      <child link="realsense_link" />
     </joint>
-    <link name="camera_link">
+    <link name="realsense_link">
       <visual>
       <origin xyz="0 ${-r410_cam_mount_from_center_offset} ${r410_cam_height/2}" rpy="${M_PI/2} 0 ${M_PI/2}"/>
@@ -56,43 +57,44 @@
       </inertial>
     </link>
+    <link name="realsense_depth_frame"/>
+    <link name="realsense_depth_optical_frame"/>
+    <link name="realsense_left_ir_frame"/>
+    <link name="realsense_left_ir_optical_frame"/>
+    <link name="realsense_right_ir_frame"/>
+    <link name="realsense_right_ir_optical_frame"/>
+    <!--<xacro:calibration_definitions child_link="$realsense_link" parent_link="${parent}" />-->
     <!-- camera depth joints and links -->
-    <joint name="camera_depth_joint" type="fixed">
+    <joint name="realsense_depth_joint" type="fixed">
       <origin xyz="${r410_cam_depth_px} ${r410_cam_depth_py} ${r410_cam_depth_pz}" rpy="0 0 0"/>
-      <parent link="camera_link"/>
-      <child link="camera_depth_frame" />
+      <parent link="realsense_link"/>
+      <child link="realsense_depth_frame" />
     </joint>
-    <link name="camera_depth_frame"/>
-    <joint name="camera_depth_optical_joint" type="fixed">
+    <joint name="realsense_depth_optical_joint" type="fixed">
       <origin xyz="0 0 0" rpy="${-M_PI/2} 0 ${-M_PI/2}" />
-      <parent link="camera_depth_frame" />
-      <child link="camera_depth_optical_frame" />
+      <parent link="realsense_depth_frame" />
+      <child link="realsense_depth_optical_frame" />
     </joint>
-    <link name="camera_depth_optical_frame"/>
     <!-- camera left IR joints and links -->
-    <joint name="camera_left_ir_joint" type="fixed">
+    <joint name="realsense_left_ir_joint" type="fixed">
       <origin xyz="0 ${r410_cam_depth_to_left_ir_offset} 0" rpy="0 0 0" />
-      <parent link="camera_depth_frame" />
-      <child link="camera_left_ir_frame" />
+      <parent link="realsense_depth_frame" />
+      <child link="realsense_left_ir_frame" />
     </joint>
-    <link name="camera_left_ir_frame"/>
-    <joint name="camera_left_ir_optical_joint" type="fixed">
+    <joint name="realsense_left_ir_optical_joint" type="fixed">
       <origin xyz="0 0 0" rpy="${-M_PI/2} 0 ${-M_PI/2}" />
-      <parent link="camera_left_ir_frame" />
-      <child link="camera_left_ir_optical_frame" />
+      <parent link="realsense_left_ir_frame" />
+      <child link="realsense_left_ir_optical_frame" />
     </joint>
-    <link name="camera_left_ir_optical_frame"/>
     <!-- camera right IR joints and links -->
-    <joint name="camera_right_ir_joint" type="fixed">
+    <joint name="realsense_right_ir_joint" type="fixed">
       <origin xyz="0 ${r410_cam_depth_to_right_ir_offset} 0" rpy="0 0 0" />
-      <parent link="camera_depth_frame" />
-      <child link="camera_right_ir_frame" />
+      <parent link="realsense_depth_frame" />
+      <child link="realsense_right_ir_frame" />
     </joint>
-    <link name="camera_right_ir_frame"/>
-    <joint name="camera_right_ir_optical_joint" type="fixed">
+    <joint name="realsense_right_ir_optical_joint" type="fixed">
       <origin xyz="0 0 0" rpy="${-M_PI/2} 0 ${-M_PI/2}" />
-      <parent link="camera_right_ir_frame" />
-      <child link="camera_right_ir_optical_frame" />
+      <parent link="realsense_right_ir_frame" />
+      <child link="realsense_right_ir_optical_frame" />
     </joint>
-    <link name="camera_right_ir_optical_frame"/>
   </xacro:macro>
 </robot>

Commit message: frame.get() does not fetch data

File: realsense_ros_camera/urdf/_r410.urdf.xacro (robot description, xacro)
@@ -28,11 +28,6 @@
     <color rgba="0.5 0.5 0.5 1"/>
   </material>
-  <xacro:macro name="sensor_r410" params="parent *origin">
+  <xacro:macro name="sensor_r410" >
     <!-- camera body, with origin at bottom screw mount -->
-    <joint name="realsense_joint" type="fixed">
-      <xacro:insert_block name="origin" />
-      <parent link="${parent}"/>
-      <child link="realsense_link" />
-    </joint>
     <link name="realsense_link">
       <visual>
@@ -59,9 +54,9 @@
     <link name="realsense_depth_frame"/>
     <link name="realsense_depth_optical_frame"/>
+    <link name="realsense_rgb_optical_frame"/>
     <link name="realsense_left_ir_frame"/>
     <link name="realsense_left_ir_optical_frame"/>
     <link name="realsense_right_ir_frame"/>
     <link name="realsense_right_ir_optical_frame"/>
-    <!--<xacro:calibration_definitions child_link="$realsense_link" parent_link="${parent}" />-->
     <!-- camera depth joints and links -->
     <joint name="realsense_depth_joint" type="fixed">
@@ -74,4 +69,9 @@
       <parent link="realsense_depth_frame" />
       <child link="realsense_depth_optical_frame" />
+    </joint>
+    <joint name="realsense_depth_optical_joint" type="fixed">
+        <origin xyz="0 0 0" rpy="${-M_PI/2} 0 ${-M_PI/2}" />
+        <parent link="realsense_depth_frame" />
+        <child link="realsense_rgb_optical_frame" />
     </joint>
     <!-- camera left IR joints and links -->
